Commit message: writes out fitness matrix

File: body.urdf (robot description, URDF)
Before this commit: robot robot, 9 links, 8 joints
Links:
- link Torso: geometry collision box size=2 1 1; visual box size=2 1 1

Commit message: writes out two fitness matrices

File: body.urdf (robot description, URDF)
Before this commit: robot robot, 9 links, 8 joints
Links:
- removed link FrontLower
- removed link FrontUpper
- added link FrontRightLower, mass 1; collision box size=0.2 0.2 1; visual box size=0.2 0.2 1
- added link FrontRightUpper, mass 1; collision box size=0.2 1 0.2; visual box size=0.2 1 0.2
Joints:
- removed joint FrontUpper_FrontLower
- removed joint Torso_FrontUpper
- added joint FrontRightUpper_FrontRightLower: type revolute, parent FrontRightUpper, child FrontRightLower, origin xyz=0 1 0 rpy=0 0 0, axis 0 1 0, limit lower=-3.14159 upper=3.14159 effort=0.0 velocity=0.0
- added joint Torso_FrontRightUpper: type revolute, parent Torso, child FrontRightUpper, origin xyz=0 0.5 1 rpy=0 0 0, axis 1 0 0, limit lower=-3.14159 upper=3.14159 effort=0.0 velocity=0.0
